Commit message: kleiner fix an den Pfaden der urdf

File: mujoco_playground/_src/locomotion/x02/x02_full_body/x02.urdf (robot description, URDF)
Before this commit: robot x2, 22 links, 21 joints
Links:
- link L_hip_yaw_link: geometry collision mesh filename=meshes/L_hip_yaw_link.STL; visual mesh filename=meshes/L_hip_yaw_link.STL
- link R_hip_yaw_link: geometry collision mesh filename=meshes/R_hip_yaw_link.STL; visual mesh filename=meshes/R_hip_yaw_link.STL
- link pelvis_link: geometry collision mesh filename=meshes/pelvis_link.STL; visual mesh filename=meshes/pelvis_link.STL

Commit message: refactoring in der full_body urdf

File: mujoco_playground/_src/locomotion/x02/x02_full_body/x02.urdf (robot description, URDF)
Before this commit: robot x2, 22 links, 21 joints
Links:
- removed link L_ankle_pitch_link
- removed link L_elbow_link
- removed link L_hip_pitch_link
- removed link L_hip_roll_link
- removed link L_hip_yaw_link
- removed link L_knee_pitch_link
- removed link L_shoulder_pitch_link
- removed link L_shoulder_roll_link
- removed link L_shoulder_yaw_link
- removed link R_ankle_pitch_link
- removed link R_elbow_link
- removed link R_hip_pitch_link
- removed link R_hip_roll_link
- removed link R_hip_yaw_link
- removed link R_knee_pitch_link
- removed link R_shoulder_pitch_link
- removed link R_shoulder_roll_link
- removed link R_shoulder_yaw_link
- added link left_ankle_pitch_link, mass 0.556154115746433; collision sphere radius=0.005; collision sphere radius=0.005
- added link left_elbow_link, mass 0.24; collision mesh filename=meshes/L_elbow_pitch_link.STL; visual mesh filename=meshes/L_elbow_pitch_link.STL
- added link left_hip_pitch_link, mass 1.332; collision mesh filename=meshes/L_hip_pitch_link.STL; visual mesh filename=meshes/L_hip_pitch_link.STL
- added link left_hip_roll_link, mass 1.562; collision mesh filename=meshes/L_hip_roll_link.STL; visual mesh filename=meshes/L_hip_roll_link.STL
- added link left_hip_yaw_link, mass 1.758; collision mesh filename=meshes/L_hip_yaw_link.STL; visual mesh filename=meshes/L_hip_yaw_link.STL
- added link left_knee_pitch_link, mass 0.847; collision mesh filename=meshes/L_knee_pitch_link.STL; visual mesh filename=meshes/L_knee_pitch_link.STL
- added link left_shoulder_pitch_link, mass 0.3; collision mesh filename=meshes/L_shoulder_pitch_link.STL; visual mesh filename=meshes/L_shoulder_pitch_link.STL
- added link left_shoulder_roll_link, mass 0.704; collision mesh filename=meshes/L_shoulder_roll_link.STL; visual mesh filename=meshes/L_shoulder_roll_link.STL
- added link left_shoulder_yaw_link, mass 0.523; collision mesh filename=meshes/L_shoulder_yaw_link.STL; visual mesh filename=meshes/L_shoulder_yaw_link.STL
- added link right_ankle_pitch_link, mass 0.556160945494453; collision sphere radius=0.005; collision sphere radius=0.005
- added link right_elbow_link, mass 0.24; collision mesh filename=meshes/R_elbow_pitch_link.STL; visual mesh filename=meshes/R_elbow_pitch_link.STL
- added link right_hip_pitch_link, mass 1.332; collision mesh filename=meshes/R_hip_pitch_link.STL; visual mesh filename=meshes/R_hip_pitch_link.STL
- added link right_hip_roll_link, mass 1.562; collision mesh filename=meshes/R_hip_roll_link.STL; visual mesh filename=meshes/R_hip_roll_link.STL
- added link right_hip_yaw_link, mass 0.907; collision mesh filename=meshes/R_hip_yaw_link.STL; visual mesh filename=meshes/R_hip_yaw_link.STL
- added link right_knee_pitch_link, mass 0.847; collision mesh filename=meshes/R_knee_pitch_link.STL; visual mesh filename=meshes/R_knee_pitch_link.STL
- added link right_shoulder_pitch_link, mass 0.3; collision mesh filename=meshes/R_shoulder_pitch_link.STL; visual mesh filename=meshes/R_shoulder_pitch_link.STL
- added link right_shoulder_roll_link, mass 0.704; collision mesh filename=meshes/R_shoulder_roll_link.STL; visual mesh filename=meshes/R_shoulder_roll_link.STL
- added link right_shoulder_yaw_link, mass 0.523; collision mesh filename=meshes/R_shoulder_yaw_link.STL; visual mesh filename=meshes/R_shoulder_yaw_link.STL
Joints:
- removed joint L_ankle_pitch_joint
- removed joint L_elbow_joint
- removed joint L_hip_pitch_joint
- removed joint L_hip_roll_joint
- removed joint L_hip_yaw_joint
- removed joint L_knee_pitch_joint
- removed joint L_shoulder_pitch_joint
- removed joint L_shoulder_roll_joint
- removed joint L_shoulder_yaw_joint
- removed joint R_ankle_pitch_joint
- removed joint R_elbow_joint
- removed joint R_hip_pitch_joint
- removed joint R_hip_roll_joint
- removed joint R_hip_yaw_joint
- removed joint R_knee_pitch_joint
- removed joint R_shoulder_pitch_joint
- removed joint R_shoulder_roll_joint
- removed joint R_shoulder_yaw_joint
- added joint left_ankle_pitch_joint: type revolute, parent left_knee_pitch_link, child left_ankle_pitch_link, origin xyz=0 0 -0.35 rpy=0 0 0, axis 0 -1 0, limit lower=-1.2217 upper=1.2217 effort=30 velocity=10
- added joint left_elbow_joint: type revolute, parent left_shoulder_yaw_link, child left_elbow_link, origin xyz=0.01 0 -0.173 rpy=0 -1.57 0, axis 0 -1 0, limit lower=-1.57 upper=0.9 effort=24 velocity=5.236
- added joint left_hip_pitch_joint: type revolute, parent left_hip_roll_link, child left_hip_pitch_link, origin xyz=0.0085 0 -0.11 rpy=0 0 0, axis 0 -1 0, limit lower=-0.5236 upper=2.0071 effort=72 velocity=9.163
- added joint left_hip_roll_joint: type revolute, parent left_hip_yaw_link, child left_hip_roll_link, origin xyz=-0.0095 0.1 -0.0474 rpy=0 0 0, axis 1 0 0, limit lower=-0.2618 upper=0.7854 effort=50 velocity=10.471975511965978
- added joint left_hip_yaw_joint: type revolute, parent pelvis_link, child left_hip_yaw_link, origin xyz=0 0 -0.06 rpy=0 0 0, axis 0 0 1, limit lower=-0.7854 upper=0.7854 effort=50 velocity=10.472
- added joint left_knee_pitch_joint: type revolute, parent left_hip_pitch_link, child left_knee_pitch_link, origin xyz=0 0 -0.35 rpy=0 0 0, axis 0 -1 0, limit lower=-2.4435 upper=0.0873 effort=60 velocity=7.3304
- added joint left_shoulder_pitch_joint: type revolute, parent torso_link, child left_shoulder_pitch_link, origin xyz=-0.01 0.14477 0.31534 rpy=0.17453 0 0, axis 0 -1 0, limit lower=-1.57 upper=3.14 effort=18 velocity=5.236
- added joint left_shoulder_roll_joint: type revolute, parent left_shoulder_pitch_link, child left_shoulder_roll_link, origin xyz=0 0.061 0 rpy=-0.17453 0 0, axis 1 0 0, limit lower=0 upper=3.141 effort=14 velocity=5.236
- added joint left_shoulder_yaw_joint: type revolute, parent left_shoulder_roll_link, child left_shoulder_yaw_link, origin xyz=0 0 -0.112 rpy=0 0 0, axis 0 0 1, limit lower=-0.66 upper=1 effort=14 velocity=5.236
- added joint right_ankle_pitch_joint: type revolute, parent right_knee_pitch_link, child right_ankle_pitch_link, origin xyz=0 0 -0.35 rpy=0 0 0, axis 0 -1 0, limit lower=-1.2217 upper=1.2217 effort=30 velocity=10
- added joint right_elbow_joint: type revolute, parent right_shoulder_yaw_link, child right_elbow_link, origin xyz=0.010039 0 -0.173 rpy=0 -1.57 0, axis 0 -1 0, limit lower=-1.57 upper=0.9 effort=24 velocity=5.236
- added joint right_hip_pitch_joint: type revolute, parent right_hip_roll_link, child right_hip_pitch_link, origin xyz=0.0085 0 -0.11 rpy=0 0 0, axis 0 -1 0, limit lower=-0.5236 upper=2.0071 effort=72 velocity=9.163
- added joint right_hip_roll_joint: type revolute, parent right_hip_yaw_link, child right_hip_roll_link, origin xyz=-0.0095 -0.1 0 rpy=0 0 0, axis -1 0 0, limit lower=-0.2618 upper=0.7854 effort=50 velocity=10.472
- added joint right_hip_yaw_joint: type revolute, parent pelvis_link, child right_hip_yaw_link, origin xyz=0 0 -0.1074 rpy=0 0 0, axis 0 0 -1, limit lower=-0.7854 upper=0.7854 effort=50 velocity=10.472
- added joint right_knee_pitch_joint: type revolute, parent right_hip_pitch_link, child right_knee_pitch_link, origin xyz=0 0 -0.35 rpy=0 0 0, axis 0 -1 0, limit lower=-2.4435 upper=0.0873 effort=60 velocity=7.3304
- added joint right_shoulder_pitch_joint: type revolute, parent torso_link, child right_shoulder_pitch_link, origin xyz=-0.01 -0.14477 0.31534 rpy=-0.17453 0 0, axis 0 -1 0, limit lower=-1.57 upper=3.14 effort=18 velocity=5.236
- added joint right_shoulder_roll_joint: type revolute, parent right_shoulder_pitch_link, child right_shoulder_roll_link, origin xyz=0 -0.061 0 rpy=0.17453 0 0, axis -1 0 0, limit lower=0 upper=3.141 effort=14 velocity=5.236
- added joint right_shoulder_yaw_joint: type revolute, parent right_shoulder_roll_link, child right_shoulder_yaw_link, origin xyz=-3.8964E-05 0 -0.112 rpy=0 0 0, axis 0 0 -1, limit lower=-0.66 upper=1 effort=14 velocity=5.236
